File: Hardware/PIR_USB.kicad_pcb (KiCad board)
At the start: 2 copper layers, 30 x 20 mm, 35 parts, among them J1 USB_C_Receptacle_USB2.0_16P, J2 Conn_01x04, J3 BS412, SW1 SW_Push, U1 STM8S003F3P, U2 CP2102N-Axx-xQFN28, U3 USBLC6-2SC6

Commit message: 250325 3
Parts:
- moved R10 14.6 mm to (56.5, 47.5), turned to 90 degrees
- moved D1 14.5 mm to (58.5, 47.5), turned to -90 degrees
- moved R16 1.80 mm to (56.5, 32.5), turned to -90 degrees
- moved D4 1.12 mm to (58.5, 32.5), turned to 90 degrees
Routing:
- net Net-(D1-A): track 1.39 -> 2.02 mm
- net Net-(D4-A): track 1.39 -> 2.02 mm
